Commit message: simulation progress

File: robomaster_description/urdf/base.urdf.xacro (robot description, xacro)
@@ -1,4 +1,4 @@
 <?xml version="1.0"?>
-  <robot xmlns:xacro="http://playerstage.sourceforge.net/gazebo/xmlschema/#xacro">
+<robot xmlns:xacro="http://playerstage.sourceforge.net/gazebo/xmlschema/#xacro">
   <xacro:include filename="led.urdf.xacro"/>
   <xacro:include filename="wheel.urdf.xacro"/>
@@ -108,3 +108,3 @@
     </material>
   </xacro:macro>
-  </robot>
+</robot>

File: robomaster_description/urdf/gimbal.urdf.xacro (robot description, xacro)
@@ -312,4 +312,4 @@
       <color rgba="0.06401 0.06401 0.06401 1.0" />
     </material>
-    </xacro:macro>
-  </robot>
+  </xacro:macro>
+</robot>
