Commit message: plugins inserted

File: robomaster_description/urdf/camera.urdf.xacro (robot description, xacro)
@@ -32,5 +32,5 @@
     <xacro:if value="${mount == 'gimbal'}">
       <joint name="${tf_prefix}camera_joint" type="fixed">
-        <origin xyz="0.0728 0.0 0.0315" rpy="0 1.5708 0"/>
+        <origin xyz="0.0728 0.0 0.0315" rpy="0 0 0"/> <!--original: rpy= 0 1.5708 0 , but this way, it looks down, through it's own skeleton-->
         <parent link="${tf_prefix}blaster_link"/>
         <child link="${tf_prefix}camera_link"/>

File: robomaster_description/urdf/gimbal.urdf.xacro (robot description, xacro)
@@ -249,5 +249,5 @@
           <mesh filename="$(find robomaster_description)/meshes/speaker.dae" scale="1.0 1.0 1.0" />
         </geometry>
-        <material name="Material #32.001" />
+        <!-- <material name="Material #32.001" /> -->
       </visual>
       <collision name="speaker_collision">

File: robomaster_description/urdf/robomaster_s1.urdf.xacro (robot description, xacro)
@@ -33,3 +33,37 @@
     </plugin>
   </gazebo>
+  <gazebo>
+    <plugin name="gazebo_ros_joint_pose_trajectory" filename="libgazebo_ros_joint_pose_trajectory.so">
+      <update_rate>20 </update_rate>
+    </plugin>
+  </gazebo>
+  <gazebo reference="camera_link">
+    <pose>0 0 0 1.57 0 0</pose>
+    <sensor type="camera" name="camera">
+      <update_rate>20</update_rate>
+      <visualize>true</visualize>
+      <camera name="cam">
+        <horizontal_fov>1.3962634</horizontal_fov>
+        <image>
+          <width>640</width>
+          <height>360</height>
+          <format>R8G8B8</format>
+        </image>
+        <clip>
+          <near>0.02</near>
+          <far>100</far>
+        </clip>
+        <noise>
+          <type>gaussian</type>
+          <mean>0.0</mean>
+          <stddev>0.007</stddev>
+        </noise>
+      </camera>
+      <plugin name="camera_controller" filename="libgazebo_ros_camera.so">
+        <frame_name>camera_optical_link</frame_name>
+        <min_depth>0.1</min_depth>
+        <max_depth>100</max_depth>
+      </plugin>
+    </sensor>
+  </gazebo>
 </robot>
