Commit message: simulation progress with ros2_control

File: robomaster_description/urdf/gimbal.urdf.xacro (robot description, xacro)
@@ -270,7 +270,4 @@
       <!-- [-25, +30] degrees -->
       <limit effort="0" velocity="0" lower="-0.5236" upper="0.4363"/>
-      <ros2_control>
-        <hardwareInterface>hardware_interface/VelocityJointInterface</hardwareInterface>
-      </ros2_control>
     </joint>
     <joint name="${tf_prefix}gimbal_left_led_joint" type="fixed">
@@ -292,5 +289,4 @@
       <limit effort="0" velocity="0" lower="-4.363" upper="4.363"/>
       <ros2_control>
-        <hardwareInterface>hardware_interface/VelocityJointInterface</hardwareInterface>
       </ros2_control>
     </joint>

File: robomaster_description/urdf/robomaster_s1.urdf.xacro (robot description, xacro)
@@ -9,4 +9,5 @@
     <xacro:property name="tf_prefix" value=""/>
   </xacro:if>
+  <xacro:include filename="control.urdf.xacro"/>
   <xacro:include filename="base.urdf.xacro"/>
   <xacro:include filename="gimbal.urdf.xacro"/>
@@ -22,32 +23,4 @@
   <xacro:add_tof index="2" tf_prefix="${tf_prefix}"/>
   <xacro:add_tof index="3" tf_prefix="${tf_prefix}"/>
-    <gazebo>
-      <plugin name="gazebo_ros_joint_state_publisher" filename="libgazebo_ros_joint_state_publisher.so">
-        <update_rate>20</update_rate>
-        <joint_name>front_left_wheel_joint</joint_name>
-        <joint_name>front_right_wheel_joint</joint_name>
-        <joint_name>rear_left_wheel_joint</joint_name>
-        <joint_name>rear_right_wheel_joint</joint_name>
-        <joint_name>blaster_joint</joint_name>
-        <joint_name>gimbal_joint</joint_name>
-        <ros>
-          <remapping>joint_states:=joint_states_p</remapping>
-        </ros>
-      </plugin>
-    </gazebo>
-    <gazebo>
-      <plugin name="gazebo_ros_joint_pose_trajectory" filename="libgazebo_ros_joint_pose_trajectory.so">
-        <update_rate>20 </update_rate>
-      </plugin>
-    </gazebo>
-  <!--
-  <gazebo>
-    <plugin name="ground_truth" filename="libgazebo_ros_p3d.so">
-      <frameName>map</frameName>
-      <bodyName>base_link</bodyName>
-      <topicName>/odom</topicName>
-      <updateRate>30.0</updateRate>
-    </plugin>
-  </gazebo> -->
   <gazebo reference="camera_link">
     <pose>0 0 0 1.57 0 0</pose>

File: robomaster_description/urdf/robomastersim.urdf (robot description, URDF)
Before this commit: robot robomaster_s1, 23 links, 22 joints
Links:
- link blaster_link: geometry collision mesh filename=/home/benko/ros2_rm/install/robomaster_description/share/ro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 scale=1.0 1.0 1.0; collision mesh filename=/home/benko/ros2_rm/install/robomaster_description/share/ro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 scale=1.0 1.0 1.0
- link camera_link: geometry visual mesh filename=/home/benko/ros2_rm/install/robomaster_description/share/ro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 scale=1.0 1.0 1.0000001
- link chassis_base_link: geometry collision mesh filename=/home/benko/ros2_rm/install/robomaster_description/share/ro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 scale=1.0 1.0 1.0; visual mesh filename=/home/benko/ros2_rm/install/robomaster_description/share/ro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 scale=1.0 1.0 1.0
- link front_hit_sensor_link: geometry visual mesh filename=($find robomaster_description)/meshes/hit_sensor.dae scale=1.0 1.0 1.0
- link front_led_link: geometry visual mesh filename=($find robomaster_description)/meshes/led.dae scale=1.0 1.0 1.0
- link front_left_wheel_link: geometry collision cylinder length=0.042 radius=0.05; visual cylinder length=0.001 radius=0.007
- link front_right_wheel_link: geometry collision cylinder length=0.042 radius=0.05; visual cylinder length=0.001 radius=0.007
- link gimbal_base_link: geometry collision mesh filename=/home/benko/ros2_rm/install/robomaster_description/share/ro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 scale=1.0 1.0 1.0; visual mesh filename=/home/benko/ros2_rm/install/robomaster_description/share/ro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 scale=1.0 1.0 1.0
- link gimbal_left_led_link: geometry visual mesh filename=/home/benko/ros2_rm/install/robomaster_description/share/ro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 scale=1.0 1.0 1.0; visual mesh filename=/home/benko/ros2_rm/install/robomaster_description/share/ro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 scale=1.0 1.0 1.0
- link gimbal_link: geometry collision mesh filename=/home/benko/ros2_rm/install/robomaster_description/share/ro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 scale=1.0 1.0 1.0; visual mesh filename=/home/benko/ros2_rm/install/robomaster_description/share/ro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 scale=1.0 1.0 1.0
- link gimbal_right_led_link: geometry visual mesh filename=/home/benko/ros2_rm/install/robomaster_description/share/ro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 scale=1.0 1.0 1.0; visual mesh filename=/home/benko/ros2_rm/install/robomaster_description/share/ro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 scale=1.0 1.0 1.0
- link intelligent_controller_link: geometry collision box size=0.108973 0.0591028 0.022915; visual mesh filename=/home/benko/ros2_rm/install/robomaster_description/share/ro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 scale=1.0 1.0 1.0
- link left_hit_sensor_link: geometry visual mesh filename=($find robomaster_description)/meshes/hit_sensor.dae scale=1.0 1.0 1.0
- link left_led_link: geometry visual mesh filename=($find robomaster_description)/meshes/led.dae scale=1.0 1.0 1.0
- link rear_hit_sensor_link: geometry visual mesh filename=($find robomaster_description)/meshes/hit_sensor.dae scale=1.0 1.0 1.0
- link rear_led_link: geometry visual mesh filename=($find robomaster_description)/meshes/led.dae scale=1.0 1.0 1.0
- link rear_left_wheel_link: geometry collision cylinder length=0.042 radius=0.05; visual cylinder length=0.001 radius=0.007
- link rear_right_wheel_link: geometry collision cylinder length=0.042 radius=0.05; visual cylinder length=0.001 radius=0.007
- link right_hit_sensor_link: geometry visual mesh filename=($find robomaster_description)/meshes/hit_sensor.dae scale=1.0 1.0 1.0
- link right_led_link: geometry visual mesh filename=($find robomaster_description)/meshes/led.dae scale=1.0 1.0 1.0
- link speaker_link: geometry collision mesh filename=/home/benko/ros2_rm/install/robomaster_description/share/ro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 scale=1.0 1.0 1.0; visual mesh filename=/home/benko/ros2_rm/install/robomaster_description/share/ro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 scale=1.0 1.0 1.0
Joints:
- joint camera_joint: origin xyz=0.0728 0.0 0.0315 rpy=0 1.5708 0 -> xyz=0.0728 0.0 0.0315 rpy=0 0 0

File: robomaster_description/urdf/wheel.urdf.xacro (robot description, xacro)
@@ -40,7 +40,4 @@
       <axis xyz="0 1.0 0"/>
       <limit effort="0" velocity="0"/>
-      <ros2_control>
-        <hardwareInterface>hardware_interface/VelocityJointInterface</hardwareInterface>
-      </ros2_control>
     </joint>
   </xacro:macro>
