Commit message: testing

File: robomaster_description/urdf/robomaster_s1.urdf.xacro (robot description, xacro)
@@ -9,5 +9,9 @@
     <xacro:property name="tf_prefix" value=""/>
   </xacro:if>
-  <xacro:include filename="control.urdf.xacro"/>
+  <link name="dummy"></link>
+  <joint name="dummy_joint" type="fixed">
+    <parent link="dummy"/>
+    <child link="base_link"/>
+  </joint>
   <xacro:include filename="base.urdf.xacro"/>
   <xacro:include filename="gimbal.urdf.xacro"/>
@@ -45,5 +49,5 @@
         </noise>
       </camera>
-      <plugin name="camera_controller" filename="libgazebo_ros_camera.so">
+      <plugin name="gazebo_camera" filename="libgazebo_ros_camera.so">
         <frame_name>camera_optical_link</frame_name>
         <min_depth>0.1</min_depth>

Commit message: using gazebo plugins instead of ros2_control

File: robomaster_description/urdf/robomaster_s1.urdf.xacro (robot description, xacro)
@@ -9,9 +9,4 @@
     <xacro:property name="tf_prefix" value=""/>
   </xacro:if>
-  <link name="dummy"></link>
-  <joint name="dummy_joint" type="fixed">
-    <parent link="dummy"/>
-    <child link="base_link"/>
-  </joint>
   <xacro:include filename="base.urdf.xacro"/>
   <xacro:include filename="gimbal.urdf.xacro"/>
@@ -56,3 +51,33 @@
     </sensor>
   </gazebo>
+  <gazebo>
+    <plugin name="robomaster_diff_drive" filename="libgazebo_ros_diff_drive.so">
+      <update_rate>30</update_rate>
+      <!-- wheels -->
+      <left_joint>front_left_wheel_joint</left_joint>
+      <right_joint>front_right_wheel_joint</right_joint>
+      <!-- kinematics -->
+      <wheel_separation>0.250</wheel_separation>
+      <wheel_diameter>0.050</wheel_diameter>
+      <!-- limits -->
+      <max_wheel_torque>20</max_wheel_torque>
+      <max_wheel_acceleration>1.0</max_wheel_acceleration>
+      <command_topic>cmd_vel</command_topic>
+      <!-- output -->
+      <publish_odom>true</publish_odom>
+      <publish_odom_tf>true</publish_odom_tf>
+      <publish_wheel_tf>false</publish_wheel_tf>
+      <odometry_topic>odom</odometry_topic>
+      <odometry_frame>odom</odometry_frame>
+      <robot_base_frame>base_link</robot_base_frame>
+    </plugin>
+    <plugin name="robomaster_joint_state" filename="libgazebo_ros_joint_state_publisher.so">
+      <ros>
+        <remapping>~/out:=joint_states</remapping>
+      </ros>
+      <update_rate>30</update_rate>
+      <joint_name>front_left_wheel_joint</joint_name>
+      <joint_name>front_right_wheel_joint</joint_name>
+    </plugin>
+  </gazebo>
 </robot>

Commit message: testing

File: robomaster_description/urdf/robomaster_s1.urdf.xacro (robot description, xacro)
@@ -22,50 +22,3 @@
   <xacro:add_tof index="2" tf_prefix="${tf_prefix}"/>
   <xacro:add_tof index="3" tf_prefix="${tf_prefix}"/>
-  <gazebo reference="camera_link">
-    <pose>0 0 0 1.57 0 0</pose>
-    <sensor type="camera" name="camera">
-      <update_rate>20</update_rate>
-      <visualize>true</visualize>
-      <camera name="cam">
-        <horizontal_fov>1.3962634</horizontal_fov>
-        <image>
-          <width>640</width>
-          <height>360</height>
-          <format>R8G8B8</format>
-        </image>
-        <clip>
-          <near>0.02</near>
-          <far>100</far>
-        </clip>
-        <noise>
-          <type>gaussian</type>
-          <mean>0.0</mean>
-          <stddev>0.007</stddev>
-        </noise>
-      </camera>
-      <plugin name="gazebo_camera" filename="libgazebo_ros_camera.so">
-        <frame_name>camera_optical_link</frame_name>
-        <min_depth>0.1</min_depth>
-        <max_depth>100</max_depth>
-      </plugin>
-    </sensor>
-  </gazebo>
-  <gazebo>
-    <plugin name="robomaster_steering" filename="libgazebo_ros_planar_move.so">
-      <commandTopic>cmd_vel</commandTopic>
-      <odometryTopic>odom</odometryTopic>
-      <odometryFrame>odom</odometryFrame>
-      <odometryRate>50.0</odometryRate>
-      <robotBaseFrame>base_link</robotBaseFrame>
-      <publishTF>false</publishTF>
-    </plugin>
-    <plugin name="robomaster_joint_state" filename="libgazebo_ros_joint_state_publisher.so">
-      <ros>
-        <remapping>~/out:=joint_states</remapping>
-      </ros>
-      <update_rate>30</update_rate>
-      <joint_name>front_left_wheel_joint</joint_name>
-      <joint_name>front_right_wheel_joint</joint_name>
-    </plugin>
-  </gazebo>
 </robot>

File: robomaster_description/urdf/robomastersim_robot1.urdf (robot description, URDF)
Before this commit: robot robomaster_1, 23 links, 22 joints
Links:
- link front_hit_sensor_link: geometry visual mesh filename=/home/benko/ros2_rm/install/robomaster_description/share/ro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 scale=1.0 1.0 1.0
- link front_led_link: geometry visual mesh filename=/home/benko/ros2_rm/install/robomaster_description/share/ro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 scale=1.0 1.0 1.0
- link left_hit_sensor_link: geometry visual mesh filename=/home/benko/ros2_rm/install/robomaster_description/share/ro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 scale=1.0 1.0 1.0
- link left_led_link: geometry visual mesh filename=/home/benko/ros2_rm/install/robomaster_description/share/ro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 scale=1.0 1.0 1.0
- link rear_hit_sensor_link: geometry visual mesh filename=/home/benko/ros2_rm/install/robomaster_description/share/ro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 scale=1.0 1.0 1.0
- link rear_led_link: geometry visual mesh filename=/home/benko/ros2_rm/install/robomaster_description/share/ro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 scale=1.0 1.0 1.0
- link right_hit_sensor_link: geometry visual mesh filename=/home/benko/ros2_rm/install/robomaster_description/share/ro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 scale=1.0 1.0 1.0
- link right_led_link: geometry visual mesh filename=/home/benko/ros2_rm/install/robomaster_description/share/ro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 scale=1.0 1.0 1.0
