Commit message: namespace corrections

File: robomaster_description/urdf/robomastersim_robot1.urdf (robot description, URDF)
Before this commit: robot robomaster_1, 23 links, 22 joints
Links:
- removed link camera_link
- added link robot1/camera_link, mass 0.001; visual mesh filename=/home/benko/ros2_rm/install/robomaster_description/share/ro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 scale=1.0 1.0 1.0000001
Joints:
- joint camera_joint: child camera_link -> robot1/camera_link
- joint camera_optical_joint: parent camera_link -> robot1/camera_link

File: robomaster_description/urdf/robomastersim_robot2.urdf (robot description, URDF)
Before this commit: robot robomaster_2, 23 links, 22 joints
Links:
- removed link camera_link
- added link robot2/camera_link, mass 0.001; visual mesh filename=/home/benko/ros2_rm/install/robomaster_description/share/ro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 scale=1.0 1.0 1.0000001
Joints:
- joint camera_joint: child camera_link -> robot2/camera_link
- joint camera_optical_joint: parent camera_link -> robot2/camera_link

Commit message: testing

File: robomaster_description/urdf/robomastersim_robot1.urdf (robot description, URDF)
Before this commit: robot robomaster_1, 23 links, 22 joints
Links:
- removed link camera_optical_link
- added link robot1/camera_optical_link, mass 0.001
Joints:
- removed joint camera_optical_joint
- added joint robot1/camera_optical_joint: type fixed, parent robot1/camera_link, child robot1/camera_optical_link, origin xyz=0.002 0.00 0.004 rpy=0.041623 0 -1.5707963267948966

File: robomaster_description/urdf/robomastersim_robot2.urdf (robot description, URDF)
Before this commit: robot robomaster_2, 23 links, 22 joints
Links:
- removed link camera_optical_link
- added link robot2/camera_optical_link, mass 0.001
Joints:
- removed joint camera_optical_joint
- added joint robot2/camera_optical_joint: type fixed, parent robot2/camera_link, child robot2/camera_optical_link, origin xyz=0.002 0.00 0.004 rpy=0.041623 0 -1.5707963267948966
